Commit message: <feat><description> add devixes.xacro for livox-lidar and realsense-D435 simulation
1. livox-lidar dependance livox_laser_simulation
2. realsense-D435 dependance realsense_ros_gazebo

File: legged_examples/legged_unitree/legged_unitree_description/urdf/robot.xacro (robot description, xacro)
@@ -2,8 +2,11 @@
 <robot xmlns:xacro="http://www.ros.org/wiki/xacro" name="robot">
     <xacro:arg name="robot_type" default="a1"/>
+    <xacro:arg name="Livox_switch" default="false"/>
+    <xacro:arg name="D435_switch" default="false"/>
     <xacro:include filename="$(find legged_unitree_description)/urdf/common/materials.xacro"/>
     <xacro:include filename="$(find legged_unitree_description)/urdf/common/leg.xacro"/>
     <xacro:include filename="$(find legged_unitree_description)/urdf/common/gazebo.xacro"/>
     <xacro:include filename="$(find legged_unitree_description)/urdf/common/imu.xacro"/>
+    <xacro:include filename="$(find legged_unitree_description)/urdf/common/devices.xacro"/>
     <xacro:include filename="$(find legged_unitree_description)/urdf/$(arg robot_type)/const.xacro"/>
     <link name="base">
@@ -29,4 +32,7 @@
         </inertial>
     </link>
+    <xacro:Devices connected_to="base" Livox_switch="$(arg Livox_switch)" D435_switch="$(arg D435_switch)">
+        <origin rpy="0 0 0" xyz="0 0 0"/>
+    </xacro:Devices>
     <xacro:IMU connected_to="base" imu_name="unitree_imu" xyz="0. 0. 0." rpy="0. 0. 0."/>
     <xacro:leg prefix="RF" mirror="-1" mirror_dae="False" front_hind="1" front_hind_dae="True">
