Commit message: <feat><add> slam simulation
1. add livox laser simulation
2. add corridor world

File: legged_examples/legged_unitree/legged_unitree_description/urdf/common/devices.xacro (robot description, xacro)
@@ -5,7 +5,7 @@
     <xacro:property name="M_PI" value="3.14159"/>
     <xacro:property name="laser_min_range" value="0.1"/>
-    <xacro:property name="laser_max_range" value="200.0"/>
+    <xacro:property name="laser_max_range" value="100.0"/>
     <xacro:property name="ros_topic" value="/livox/lidar"/>
-    <xacro:property name="samples" value="24000"/>
+    <xacro:property name="samples" value="12000"/>
     <xacro:property name="downsample" value="1"/>
     <xacro:macro name="Devices" params="connected_to *origin Livox_switch:=false D435_switch:=false">
@@ -37,5 +37,5 @@
                 <geometry>
                     <box size="0.18 0.24 0.08"/>
-                    <!-- <mesh filename="package://legged_unitree_description/meshes/devices/drives_link.STL" /> -->
+                    <mesh filename="package://legged_unitree_description/meshes/devices/drives_link.STL" />
                 </geometry>
             </collision>
@@ -60,5 +60,5 @@
                 <origin xyz="0 0 0" rpy="0 0 0" />
                 <geometry>
-                    <!-- <mesh filename="package://legged_unitree_description/meshes/devices/mid360_link.STL" /> -->
+                    <mesh filename="package://legged_unitree_description/meshes/devices/mid360_link.STL" />
                 </geometry>
             </collision>
@@ -70,8 +70,8 @@
             <axis xyz="0 0 0" />
         </joint>
-        <xacro:macro name="Livox_Mid_gazebo_sensor" params="visualize:=True update_rate:=10 resolution:=0.002 noise_mean:=0.0 noise_stddev:=0.01 name:=livox">
+        <xacro:macro name="Livox_Mid_gazebo_sensor" params="visualize:=True update_rate:=10 resolution:=0.01 noise_mean:=0.0 noise_stddev:=0.01 name:=mid360">
             <gazebo reference="mid360_link">
                 <sensor type="ray" name="laser_${name}">
-                    <pose>0 0 0 0 0 0</pose>
+                    <pose>0.067374 0 0.14292 0 0 0</pose>
                     <visualize>${visualize}</visualize>
                     <update_rate>${update_rate}</update_rate>

File: legged_examples/legged_unitree/legged_unitree_description/urdf/robot.xacro (robot description, xacro)
@@ -4,4 +4,8 @@
     <xacro:arg name="Livox_switch" default="false"/>
     <xacro:arg name="D435_switch" default="false"/>
+    <xacro:arg name="Devices_switch" default="false"/>
+    <xacro:property name="Livox_switch_flag" value="$(arg Livox_switch)"/>
+    <xacro:property name="D435_switch_flag" value="$(arg D435_switch)"/>
+    <xacro:property name="Devices_switch_flag" value="$(arg Devices_switch)"/>
     <xacro:include filename="$(find legged_unitree_description)/urdf/common/materials.xacro"/>
     <xacro:include filename="$(find legged_unitree_description)/urdf/common/leg.xacro"/>
@@ -32,7 +36,9 @@
         </inertial>
     </link>
-    <!-- <xacro:Devices connected_to="base" Livox_switch="$(arg Livox_switch)" D435_switch="$(arg D435_switch)">
-        <origin rpy="0 0 0" xyz="0 0 0"/>
-    </xacro:Devices> -->
+    <xacro:if value="${Devices_switch_flag == True}">
+        <xacro:Devices connected_to="base" Livox_switch="${Livox_switch_flag}" D435_switch="${D435_switch_flag}">
+            <origin rpy="0 0 0" xyz="0 0 0"/>
+        </xacro:Devices>
+    </xacro:if>
     <xacro:IMU connected_to="base" imu_name="unitree_imu" xyz="0. 0. 0." rpy="0. 0. 0."/>
     <xacro:leg prefix="RF" mirror="-1" mirror_dae="False" front_hind="1" front_hind_dae="True">

Commit message: <feat><description> modify for simulation

File: legged_examples/legged_unitree/legged_unitree_description/urdf/common/devices.xacro (robot description, xacro)
@@ -37,5 +37,5 @@
                 <geometry>
                     <box size="0.18 0.24 0.08"/>
-                    <mesh filename="package://legged_unitree_description/meshes/devices/drives_link.STL" />
+                    <!-- <mesh filename="package://legged_unitree_description/meshes/devices/drives_link.STL" /> -->
                 </geometry>
             </collision>
@@ -60,5 +60,6 @@
                 <origin xyz="0 0 0" rpy="0 0 0" />
                 <geometry>
-                    <mesh filename="package://legged_unitree_description/meshes/devices/mid360_link.STL" />
+                    <box size="0.0 0.0 0.0"/>
+                    <!-- <mesh filename="package://legged_unitree_description/meshes/devices/mid360_link.STL" /> -->
                 </geometry>
             </collision>
@@ -135,4 +136,5 @@
                 <origin xyz="0 0 0" rpy="0 0 0" />
                 <geometry>
+                    <box size="0.0 0.0 0.0"/>
                     <!-- <mesh filename="package://legged_unitree_description/meshes/devices/cam_bracker_link.STL" /> -->
                 </geometry>

File: legged_examples/legged_unitree/legged_unitree_description/urdf/robot.xacro (robot description, xacro)
@@ -5,7 +5,9 @@
     <xacro:arg name="D435_switch" default="false"/>
     <xacro:arg name="Devices_switch" default="false"/>
+    <xacro:arg name="Laser_switch" default="false"/>
     <xacro:property name="Livox_switch_flag" value="$(arg Livox_switch)"/>
     <xacro:property name="D435_switch_flag" value="$(arg D435_switch)"/>
     <xacro:property name="Devices_switch_flag" value="$(arg Devices_switch)"/>
+    <xacro:property name="Laser_switch_flag" value="$(arg Laser_switch)"/>
     <xacro:include filename="$(find legged_unitree_description)/urdf/common/materials.xacro"/>
     <xacro:include filename="$(find legged_unitree_description)/urdf/common/leg.xacro"/>
@@ -36,4 +38,63 @@
         </inertial>
     </link>
+    <xacro:if value="${Laser_switch_flag == True}">
+        <joint name="hokuyo_joint" type="fixed">
+            <origin rpy="0 0 0" xyz="0.0 0.0 0.105"/>
+            <parent link="base"/>
+            <child link="hokuyo_frame"/>
+        </joint>
+        <link name="hokuyo_frame">
+            <inertial>
+                <mass value="0.270"/>
+                <origin rpy="0 0 0" xyz="0 0 0"/>
+                <inertia ixx="2.632e-4" ixy="0" ixz="0" iyy="2.632e-4" iyz="0" izz="1.62e-4"/>
+            </inertial>
+            <visual>
+                <origin rpy="0 0 0" xyz="0 0 0"/>
+                <geometry>
+                    <mesh filename="package://hector_sensors_description/meshes/hokuyo_utm30lx/hokuyo_utm_30lx.dae"/>
+                </geometry>
+            </visual>
+            <collision>
+                <origin rpy="0 0 0" xyz="0 0 -0.0115"/>
+                <geometry>
+                    <box size="0.058 0.058 0.087"/>
+                    <!--<mesh filename="package://hector_sensors_description/meshes/hokuyo_utm30lx/hokuyo_utm_30lx.stl"/>-->
+                </geometry>
+            </collision>
+        </link>
+        <gazebo reference="hokuyo_frame">
+            <sensor name="hokuyo" type="ray">
+                <always_on>true</always_on>
+                <update_rate>30</update_rate>
+                <pose>0 0 0 0 0 0</pose>
+                <visualize>false</visualize>
+                <ray>
+                    <scan>
+                        <horizontal>
+                            <samples>1040</samples>
+                            <resolution>1</resolution>
+                            <min_angle>2.26892802759</min_angle>
+                            <max_angle>-2.26892802759</max_angle>
+                        </horizontal>
+                    </scan>
+                    <range>
+                        <min>0.2</min>
+                        <max>30.0</max>
+                        <resolution>0.01</resolution>
+                    </range>
+                    <noise>
+                        <type>gaussian</type>
+                        <mean>0.0</mean>
+                        <stddev>0.004</stddev>
+                    </noise>
+                </ray>
+                <plugin filename="libgazebo_ros_laser.so" name="gazebo_ros_hokuyo_controller">
+                    <topicName>scan</topicName>
+                    <frameName>hokuyo_frame</frameName>
+                </plugin>
+            </sensor>
+        </gazebo>
+    </xacro:if>
     <xacro:if value="${Devices_switch_flag == True}">
         <xacro:Devices connected_to="base" Livox_switch="${Livox_switch_flag}" D435_switch="${D435_switch_flag}">
